File: metademo.kicad_sch (KiCad schematic)
At the start: 22 parts, among them IC1 MAX6817EUT+T, IC2 TLV1117LV33DCYR, J1 CONBNC001, J2 CONBNC001, J3 CONBNC001, J4 CONBNC001, J5 Conn_01x01_Pin, J6 Conn_01x01_Pin, U1 SN74LVC2G74DCUR

Commit message: updates
Parts:
- removed J5: Conn_01x01_Pin, Connector_Wire:SolderWire-2.5sqmm_1x01_D2.4mm_OD4.4mm, symbol Connector:Conn_01x01_Pin
